Commit message: updates

File: src/touch_pack/urdf/touch_tool_square_20x20.urdf (robot description, URDF)
Before this commit: robot touch_tool_tcp, 5 links, 4 joints
Links:
- link force_sensor_link: mass 0.400 -> 0.800; geometry collision box size=0.0508 0.0191 0.0762; collision cylinder length=0.008 radius=0.03175
Joints:
- joint force_sensor_attach: origin xyz=0 0 0 rpy=0 0 -1.5708 -> xyz=0 0 0 rpy=0 0 0
- joint touch_tool_attach: origin xyz=0.055 0 0.028 rpy=0 0 1.5708 -> xyz=0 0 0.0922 rpy=0 0 0
